File: Final Project - Jay J Gurung/Arpeggio Machine - Final Project - Jay J Gurung/Arpeggio Machine - Final Project - Jay J Gurung.kicad_sch (KiCad schematic)
At the start: 0 parts

Commit message: update kicad
update
Parts:
- added J1: Speaker, TerminalBlock_Phoenix:TerminalBlock_Phoenix_MKDS-1,5-2-5.08_1x02_P5.08mm_Horizontal, symbol Connector:Conn_01x02_Pin
- added J2: AMP_PAM8302, Connector_PinHeader_2.54mm:PinHeader_1x05_P2.54mm_Vertical, symbol Connector:Conn_01x05_Pin
- added RV1: BPM_POT, Potentiometer_THT:Potentiometer_Alpha_RD901F-40-00D_Single_Vertical, symbol Device:R_Potentiometer
- added RV2: NOTE_LEN_POT, Potentiometer_THT:Potentiometer_Alpha_RD901F-40-00D_Single_Vertical, symbol Device:R_Potentiometer
- added RV3: ROOT_POT, Potentiometer_THT:Potentiometer_Alpha_RD901F-40-00D_Single_Vertical, symbol Device:R_Potentiometer
- added RV4: VOLUME_SLIDE_POT, Potentiometer_THT:Potentiometer_Bourns_PTA4543_Single_Slide, symbol Device:R_Potentiometer
- added SW1: BTN_APPLY_ROOT, symbol Switch:SW_Push
- added SW2: SW_PLAY_MODE, Connector_JST:JST_XH_B3B-XH-A_1x03_P2.50mm_Vertical, symbol Switch:SW_SPDT
- added SW3: SW_WAVE_TYPE, Connector_JST:JST_XH_B3B-XH-A_1x03_P2.50mm_Vertical, symbol Switch:SW_SPDT
- added SW4: SW_SCALE_MODE, Connector_JST:JST_XH_B3B-XH-A_1x03_P2.50mm_Vertical, symbol Switch:SW_SPDT
- added U1: ESP32-S3-DevKitC, PCM_Espressif:ESP32-S3-DevKitC, symbol Espressif:ESP32-S3-DevKitC
Connections:
- new net: U1.1 (3V3), U1.2 (3V3)
- new net: U1.22 (GND), U1.23 (GND), U1.24 (GND), U1.44 (GND)
Other:
- company: (none) -> AAGO STUDIO INC
- title: (none) -> Arpeggio Machine - Final Project - Jay J Gurung
